File: psu.kicad_sch (KiCad schematic)
At the start: 30 parts, among them J3 Screw_Terminal_01x03, Q1 BT136-800, T2 POE30P-33L, U2 PC817, U3 TL431DBZ, U4 MOC3021M, U5 VIPer22AS, U6 PC817

Commit message: schematic completed:
Connections:
- net ZV signal out renamed ZVC signal out
Other:
- moved on the sheet: R9
Changed lines of the file:
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@@
+    (stroke (width 0) (type default))
+  )
+  (wire (pts (xy 128.905 95.25) (xy 132.08 95.25))
     (stroke (width 0) (type default))
   )
@@
     (stroke (width 0) (type default))
   )
-  (wire (pts (xy 118.11 93.98) (xy 118.11 99.06))
+  (wire (pts (xy 118.11 95.25) (xy 118.11 99.06))
     (stroke (width 0) (type default))
   )
@@
     (stroke (width 0) (type default))
   )
-  (wire (pts (xy 129.54 93.98) (xy 132.08 93.98))
-    (stroke (width 0) (type default))
-  )
   (wire (pts (xy 157.48 87.63) (xy 157.48 88.9))
     (stroke (width 0) (type default))
@@
     (stroke (width 0) (type default))
   )
-  (wire (pts (xy 118.11 93.98) (xy 121.92 93.98))
+  (wire (pts (xy 118.11 95.25) (xy 121.285 95.25))
     (stroke (width 0) (type default))
   )
@@
     (effects (font (size 1.27 1.27)) (justify left bottom))
   )
-  (label "3.3V" (at 132.08 93.98 0) (fields_autoplaced)
+  (label "3.3V" (at 132.08 95.25 0) (fields_autoplaced)
     (effects (font (size 1.27 1.27)) (justify left bottom))
   )
@@
     (effects (font (size 1.27 1.27)) (justify left))
   )
-  (hierarchical_label "ZV signal out" (shape output) (at 121.92 99.06 0) (fields_autoplaced)
+  (hierarchical_label "ZVC signal out" (shape output) (at 121.92 99.06 0) (fields_autoplaced)
     (effects (font (size 1.27 1.27)) (justify left))
   )
@@
     )
   )
-  (symbol (lib_id "Device:R") (at 125.73 93.98 270) (unit 1)
-    (in_bom yes) (on_board yes) (dnp no)
-    (property "Reference" "R9" (at 125.73 93.98 90)
-      (effects (font (size 1.27 1.27)))
-    )
-    (property "Value" "1.5k" (at 125.73 91.44 90)
-      (effects (font (size 1.27 1.27)))
-    )
-    (property "Footprint" "Resistor_SMD:R_0402_1005Metric" (at 125.73 92.202 90)
-      (effects (font (size 1.27 1.27)) hide)
-    )
-    (property "Datasheet" "~" (at 125.73 93.98 0)
-      (effects (font (size 1.27 1.27)) hide)
-    )
+  (symbol (lib_id "Device:R") (at 125.095 95.25 270) (unit 1)
+    (in_bom yes) (on_board yes) (dnp no)
+    (property "Reference" "R9" (at 125.095 95.25 90)
+      (effects (font (size 1.27 1.27)))
+    )
+    (property "Value" "1.5k" (at 125.095 92.71 90)
+      (effects (font (size 1.27 1.27)))
+    )
+    (property "Footprint" "Resistor_SMD:R_0402_1005Metric" (at 125.095 93.472 90)
+      (effects (font (size 1.27 1.27)) hide)
+    )
+    (property "Datasheet" "~" (at 125.095 95.25 0)
+      (effects (font (size 1.27 1.27)) hide)
+    )
